File: Power controller/Design/Power/Power.sch (KiCad schematic (older format))
At the start: 28 parts

Commit message: Added ICSP, assigned footprints
Parts:
- removed F?: Fuse, symbol Device:Fuse
- removed Q? (x3): IRF6613, Package_DirectFET:DirectFET_MT, symbol Transistor_FET:IRF6613
- added C4: 3.9n, Capacitor_SMD:C_0805_2012Metric_Pad1.15x1.40mm_HandSolder, symbol Device:C_Small
- added C8: 100n, Capacitor_SMD:C_0805_2012Metric_Pad1.15x1.40mm_HandSolder, symbol Device:C_Small
- added F1: 0154010.DR, SamacSys_Parts:0154001.DRT, symbol SamacSys_Parts:0154010.DR
- added J2: Conn_02x03_Odd_Even, Connector_PinHeader_2.54mm:PinHeader_2x03_P2.54mm_Vertical, symbol Connector_Generic:Conn_02x03_Odd_Even
- added J3: Conn_01x02, Connector_PinHeader_2.54mm:PinHeader_1x02_P2.54mm_Vertical, symbol Connector_Generic:Conn_01x02
- added L2: 10u, Inductor_SMD:L_1210_3225Metric_Pad1.42x2.65mm_HandSolder, symbol Device:L_Small
- added Q1, Q2, Q3: IRF7403, Package_SO:SOIC-8_3.9x4.9mm_P1.27mm, symbol Transistor_FET:IRF7403
- added R1: 6.8k, Resistor_SMD:R_0805_2012Metric_Pad1.15x1.40mm_HandSolder, symbol Device:R_Small
- C1, C2, C3, C5, C6, C7: renamed from C?; footprint (none) -> Capacitor_SMD:C_0805_2012Metric_Pad1.15x1.40mm_HandSolder
- IC1: renamed from IC?; footprint SOIC127P600X170-9N -> SamacSys_Parts:SOIC127P600X170-9N; symbol SamacSys_Parts:MP2307DN-LF-Z -> Power-rescue:MP2307DN-LF-Z-SamacSys_Parts
- IC2: renamed from IC?; footprint SON40P300X300X80-15N -> SamacSys_Parts:SON40P300X300X80-15N; symbol SamacSys_Parts:MAX17261METD+ -> Power-rescue:MAX17261METD+-SamacSys_Parts
- J1: renamed from J?; footprint (none) -> Connector_Molex:Molex_Nano-Fit_105313-xx02_1x02_P2.50mm_Horizontal
- L1: renamed from L?; footprint (none) -> Inductor_SMD:L_Vishay_IHLP-2525
- R2, R3, R4, R5, R6, R7: renamed from R?; footprint (none) -> Resistor_SMD:R_0805_2012Metric_Pad1.15x1.40mm_HandSolder
- Y1: renamed from Y?; footprint (none) -> Crystal:Crystal_SMD_TXC_7A-2Pin_5x3.2mm
- gave numbers to parts that had none: 7
Connections:
- net +5V: now also J3.2 (Pin_2)
- net BGND: now also J1.1 (Pin_1), R1.2; no longer J1.2 (Pin_2)
- net GND: now also U1.21 (GND), U1.33 (GND), U1.5 (GND), C8.1, J2.6 (Pin_6), Q1.1 (S), Q1.2 (S), Q1.3 (S), Q2.1 (S), Q2.2 (S), Q2.3 (S), Q3.1 (S), Q3.2 (S), Q3.3 (S)
- net VBAT: now also F1.2
- net MOSI: now reaches U1.15 (PB3)
- net MOSI: now also J2.4 (Pin_4)
- net MISO: now reaches U1.16 (PB4)
- net MISO: now also J2.1 (Pin_1)
- net SCK: now reaches U1.17 (PB5)
- net SCK: now also J2.3 (Pin_3)
- net at U1.18 (AVCC): now also C8.2, L2.2
- net RESET: now reaches U1.29 (~RESET~/PC6)
- net RESET: now also J2.5 (Pin_5)
- net at U1.4 (VCC): now also L2.1
- net at U5.1 (IP+), U5.2 (IP+): now also Q1.5 (D), Q1.6 (D), Q1.7 (D), Q1.8 (D)
- net at U2.5 (~OUT): now also Q1.4 (G)
- net at U6.1 (IP+), U6.2 (IP+): now also Q2.5 (D), Q2.6 (D), Q2.7 (D), Q2.8 (D)
- net at U3.5 (~OUT): now also Q2.4 (G)
- net at U7.1 (IP+), U7.2 (IP+): now also Q3.5 (D), Q3.6 (D), Q3.7 (D), Q3.8 (D)
- net at U4.5 (~OUT): now also Q3.4 (G)
- net at IC1.5 (FB), R2.1, R3.2: now also IC1.6 (COMP), C4.1
- new net: F1.1, J1.2 (Pin_2)
- new net: C4.2, R1.1
- new net +5V_MCU: J2.2 (Pin_2), J3.1 (Pin_1)

Commit message: Removed fuel gauge, grouped PCB
Parts:
- removed C7: 0.47u, Capacitor_SMD:C_0805_2012Metric_Pad1.15x1.40mm_HandSolder, symbol Device:C_Small
- removed IC2: MAX17261METD+, SamacSys_Parts:SON40P300X300X80-15N, symbol Power-rescue:MAX17261METD+-SamacSys_Parts
- removed R7: 200k, Resistor_SMD:R_0805_2012Metric_Pad1.15x1.40mm_HandSolder, symbol Device:R_Small
- added Q4, Q5: IRF7403, Package_SO:SOIC-8_3.9x4.9mm_P1.27mm, symbol Transistor_FET:IRF7403
- F1: symbol SamacSys_Parts:0154010.DR -> Power-rescue:0154010.DR-SamacSys_Parts
- IC1: symbol Power-rescue:MP2307DN-LF-Z-SamacSys_Parts -> Power-rescue:MP2307DN-LF-Z-SamacSys_Parts-Power-rescue
- R5: value 5m -> 4k7
- R6: value 1.8M -> 4k7
Connections:
- net GND: no longer R5.1
- net VBAT: no longer R6.2
- net SDA: now reaches U1.27 (PC4)
- net SDA: now also R5.1, Q4.5 (D), Q4.6 (D), Q4.7 (D), Q4.8 (D)
- net SCL: now reaches U1.28 (PC5)
- net SCL: now also R6.1, Q5.5 (D), Q5.6 (D), Q5.7 (D), Q5.8 (D)
- net 5V: now reaches R5.2
- net 5V: now also R6.2
- new net 3V3: Q4.4 (G), Q5.4 (G)
- new net SCL3: Q5.1 (S), Q5.2 (S), Q5.3 (S)
- new net SDA3: Q4.1 (S), Q4.2 (S), Q4.3 (S)
Other:
- note removed: "Fuel gauge"
Changed lines of the file:
@@
 	8150 2850 8150 2900
-$Comp
-L Power-rescue:MAX17261METD+-SamacSys_Parts IC2
-U 1 1 5C2CE787
-P 7750 4850
-F 0 "IC2" H 8350 5115 50  0000 C CNN
-F 1 "MAX17261METD+" H 8350 5024 50  0000 C CNN
-F 2 "SamacSys_Parts:SON40P300X300X80-15N" H 8800 4950 50  0001 L CNN
-F 3 "https://datasheets.maximintegrated.com/en/ds/MAX17261.pdf" H 8800 4850 50  0001 L CNN
-F 4 "Battery Management 5A Multi-Cell Fuel Gauge with ModelGauge m5 EZ" H 8800 4750 50  0001 L CNN "Description"
-F 5 "0.8" H 8800 4650 50  0001 L CNN "Height"
-F 6 "Maxim Integrated" H 8800 4550 50  0001 L CNN "Manufacturer_Name"
-F 7 "MAX17261METD+" H 8800 4450 50  0001 L CNN "Manufacturer_Part_Number"
-F 8 "" H 8800 4350 50  0001 L CNN "RS Part Number"
-F 9 "" H 8800 4250 50  0001 L CNN "RS Price/Stock"
-F 10 "700-MAX17261METD+" H 8800 4150 50  0001 L CNN "Mouser Part Number"
-F 11 "https://www.mouser.com/Search/Refine.aspx?Keyword=700-MAX17261METD%2B" H 8800 4050 50  0001 L CNN "Mouser Price/Stock"
-	1    7750 4850
-	1    0    0    -1
-$EndComp
 $Comp
 L Sensor_Current:ACS723xLCTR-10AU U5
@@
 Wire Wire Line
 	8750 3250 8750 3150
-$Comp
-L Device:R_Small R6
-U 1 1 5C2D46A9
-P 9550 5350
-F 0 "R6" H 9609 5396 50  0000 L CNN
-F 1 "1.8M" H 9609 5305 50  0000 L CNN
-F 2 "Resistor_SMD:R_0805_2012Metric_Pad1.15x1.40mm_HandSolder" H 9550 5350 50  0001 C CNN
-F 3 "~" H 9550 5350 50  0001 C CNN
-	1    9550 5350
-	1    0    0    -1
-$EndComp
-$Comp
-L Device:R_Small R7
-U 1 1 5C2D475F
-P 9850 5250
-F 0 "R7" V 10046 5250 50  0000 C CNN
-F 1 "200k" V 9955 5250 50  0000 C CNN
-F 2 "Resistor_SMD:R_0805_2012Metric_Pad1.15x1.40mm_HandSolder" H 9850 5250 50  0001 C CNN
-F 3 "~" H 9850 5250 50  0001 C CNN
-	1    9850 5250
-	0    -1   -1   0
-$EndComp
-Text GLabel 10000 5250 2    50   Input ~ 0
-BGND
-Text GLabel 9550 5500 3    50   Input ~ 0
-VBAT
-Wire Wire Line
-	9950 5250 10000 5250
-$Comp
-L Device:C_Small C7
-U 1 1 5C2D6508
-P 9200 5150
-F 0 "C7" V 8971 5150 50  0000 C CNN
-F 1 "0.47u" V 9062 5150 50  0000 C CNN
-F 2 "Capacitor_SMD:C_0805_2012Metric_Pad1.15x1.40mm_HandSolder" H 9200 5150 50  0001 C CNN
-F 3 "~" H 9200 5150 50  0001 C CNN
-	1    9200 5150
-	0    1    1    0
-$EndComp
-Wire Wire Line
-	8950 5150 9100 5150
-Wire Wire Line
-	8950 5250 9550 5250
-Connection ~ 9550 5250
-Wire Wire Line
-	9550 5250 9750 5250
-Wire Wire Line
-	9550 5500 9550 5450
-Text GLabel 9350 5150 2    50   Input ~ 0
-BGND
-Wire Wire Line
-	9350 5150 9300 5150
-Text GLabel 7700 4850 0    50   Input ~ 0
-+5V
-Text GLabel 7700 5350 0    50   Input ~ 0
-+5V
-Wire Wire Line
-	7700 5350 7750 5350
-Wire Wire Line
-	7700 4850 7750 4850
-$Comp
-L Device:R_Small R5
-U 1 1 5C2DC9F7
-P 7750 5650
-F 0 "R5" H 7809 5696 50  0000 L CNN
-F 1 "5m" H 7809 5605 50  0000 L CNN
-F 2 "Resistor_SMD:R_0805_2012Metric_Pad1.15x1.40mm_HandSolder" H 7750 5650 50  0001 C CNN
-F 3 "~" H 7750 5650 50  0001 C CNN
-	1    7750 5650
-	1    0    0    -1
-$EndComp
-Wire Wire Line
-	7750 5750 7750 5950
-Wire Wire Line
-	7750 5950 8350 5950
-Wire Wire Line
-	8350 5950 8950 5950
-Wire Wire Line
-	8950 5950 8950 5450
-Connection ~ 8350 5950
-Wire Wire Line
-	8950 5450 8950 5350
-Connection ~ 8950 5450
-Wire Wire Line
-	7750 5550 7750 5450
-Text GLabel 7700 5450 0    50   Input ~ 0
-GND
-Wire Wire Line
-	7700 5450 7750 5450
-Connection ~ 7750 5450
-Text GLabel 9050 4600 1    50   Input ~ 0
-ALERT
-Wire Wire Line
-	8950 5050 9050 5050
-Wire Wire Line
-	9050 5050 9050 4600
 Text GLabel 2150 3150 2    50   Input ~ 0
 ALERT
@@
 Text Notes 8050 750  2    118  ~ 0
 Power & control
-Text Notes 8450 4450 2    118  ~ 0
-Fuel gauge
 $Comp
 L Connector_Generic:Conn_01x02 J1
@@
 VBAT
 $Comp
-L Power-rescue:MP2307DN-LF-Z-SamacSys_Parts IC1
+L Power-rescue:MP2307DN-LF-Z-SamacSys_Parts-Power-rescue IC1
 U 1 1 5C3044AC
 P 4300 1200
@@
 	3850 2450 3950 2450
 $Comp
-L SamacSys_Parts:0154010.DR F1
+L Power-rescue:0154010.DR-SamacSys_Parts F1
 U 1 1 5C3D91AA
 P 4050 2350
@@
 Wire Wire Line
 	2150 2650 2100 2650
+$Comp
+L Device:R_Small R5
+U 1 1 5C7E5782
+P 2900 3350
+F 0 "R5" H 2841 3304 50  0000 R CNN
+F 1 "4k7" H 2841 3395 50  0000 R CNN
+F 2 "Resistor_SMD:R_0805_2012Metric_Pad1.15x1.40mm_HandSolder" H 2900 3350 50  0001 C CNN
+F 3 "~" H 2900 3350 50  0001 C CNN
+	1    2900 3350
+	-1   0    0    1
+$EndComp
+$Comp
+L Device:R_Small R6
+U 1 1 5C7E581A
+P 3250 3350
+F 0 "R6" H 3191 3304 50  0000 R CNN
+F 1 "4k7" H 3191 3395 50  0000 R CNN
+F 2 "Resistor_SMD:R_0805_2012Metric_Pad1.15x1.40mm_HandSolder" H 3250 3350 50  0001 C CNN
+F 3 "~" H 3250 3350 50  0001 C CNN
+	1    3250 3350
+	-1   0    0    1
+$EndComp
+Wire Wire Line
+	2900 3250 3100 3250
+Text GLabel 2900 3550 3    50   Input ~ 0
+SDA
+Text GLabel 3250 3550 3    50   Input ~ 0
+SCL
+Wire Wire Line
+	2900 3450 2900 3550
+Text GLabel 3100 3100 1    50   Input ~ 0
+5V
+Wire Wire Line
+	3100 3100 3100 3250
+Wire Wire Line
+	3250 3450 3250 3550
+Wire Wire Line
+	3250 3250 3100 3250
+Connection ~ 3100 3250
+$Comp
+L Transistor_FET:IRF7403 Q4
+U 1 1 5C8128D4
+P 4350 3450
+F 0 "Q4" V 4600 3450 50  0000 C CNN
+F 1 "IRF7403" V 4691 3450 50  0000 C CNN
+F 2 "Package_SO:SOIC-8_3.9x4.9mm_P1.27mm" H 4550 3350 50  0001 L CNN
+F 3 "https://www.infineon.com/dgdl/irf7403pbf.pdf?fileId=5546d462533600a4015355fa23541b9c" H 4250 3450 50  0001 L CNN
+	1    4350 3450
+	0    1    1    0
+$EndComp
+$Comp
+L Transistor_FET:IRF7403 Q5
+U 1 1 5C812998
+P 5200 3450
+F 0 "Q5" V 5450 3450 50  0000 C CNN
+F 1 "IRF7403" V 5541 3450 50  0000 C CNN
+F 2 "Package_SO:SOIC-8_3.9x4.9mm_P1.27mm" H 5400 3350 50  0001 L CNN
+F 3 "https://www.infineon.com/dgdl/irf7403pbf.pdf?fileId=5546d462533600a4015355fa23541b9c" H 5100 3450 50  0001 L CNN
+	1    5200 3450
+	0    1    1    0
+$EndComp
+Text GLabel 4650 3550 2    50   Input ~ 0
+SDA
+Text GLabel 5500 3550 2    50   Input ~ 0
+SCL
+Text GLabel 4800 3150 1    50   Input ~ 0
+3V3
+Wire Wire Line
+	4350 3250 4800 3250
+Wire Wire Line
+	4800 3150 4800 3250
+Connection ~ 4800 3250
+Wire Wire Line
+	4800 3250 5200 3250
+Wire Wire Line
+	4550 3550 4650 3550
+Wire Wire Line
+	5400 3550 5500 3550
+Text GLabel 4050 3550 0    50   Input ~ 0
+SDA3
+Text GLabel 5000 3700 0    50   Input ~ 0
+SCL3
+Wire Wire Line
+	5000 3700 5000 3550
+Wire Wire Line
+	4050 3550 4150 3550
+Text GLabel 2150 2450 2    50   Input ~ 0
+SDA
+Text GLabel 2150 2550 2    50   Input ~ 0
+SCL
+Wire Wire Line
+	2100 2550 2150 2550
+Wire Wire Line
+	2100 2450 2150 2450
 $EndSCHEMATC
